Commit message: updated panda config, and panda and mycobot urdf

File: models/elephant_description/mycobot_280_pi.urdf (robot description, URDF)
Before this commit: robot firefighter, 8 links, 7 joints
Links:
- link g_base: mass None -> 0.2
- link joint1: mass None -> 0.2
- link joint2: mass None -> 0.2
- link joint3: mass None -> 0.2
- link joint4: mass None -> 0.2
- link joint5: mass None -> 0.2
- link joint6: mass None -> 0.2
- link joint6_flange: mass None -> 0.05

File: models/panda_description/panda.urdf (robot description, URDF)
Before this commit: robot panda, 9 links, 8 joints
Joints:
- joint panda_joint4: limit lower=-3.0718 upper=-0.0698 effort=87 velocity=2.1750 -> lower=0.0 upper=3.002 effort=87 velocity=2.1750

Commit message: updating urdf and config for elephant to align with real better

File: models/elephant_description/mycobot_280_pi.urdf (robot description, URDF)
Before this commit: robot firefighter, 8 links, 7 joints
Links:
- added link gripper
- added link robot_base
- link g_base: mass 0.2 -> None; geometry 
Joints:
- added joint joint6output_to_gripper: type fixed, parent joint6_flange, child gripper, origin xyz=0 0 0.1 rpy=0 0 -0.5236
- added joint robot_base_to_g_base: type fixed, parent robot_base, child g_base, origin xyz=0 0 0.003 rpy=0 0 0
- joint g_base_to_joint1: origin xyz=0 0 0 rpy=0 0 0 -> xyz=0 0 0.026 rpy=0 0 0
