Commit message: cleaned urdf model  and  added new urdf for pinocchio

File: models/summit_xl_arm_description/summit_xl_complete_pin.urdf (robot description, URDF)
Before this commit: robot summit_xl, 24 links, 23 joints
Joints:
- joint robot_back_left_wheel_joint: limit effort=100 velocity=100 -> lower=-1000000 upper=1000000 effort=100 velocity=100; type continuous -> revolute
- joint robot_back_right_wheel_joint: limit effort=100 velocity=100 -> lower=-1000000 upper=1000000 effort=100 velocity=100; type continuous -> revolute
- joint robot_front_left_wheel_joint: limit effort=100 velocity=100 -> lower=-1000000 upper=1000000 effort=100 velocity=100; type continuous -> revolute
- joint robot_front_right_wheel_joint: limit effort=100 velocity=100 -> lower=-1000000 upper=1000000 effort=100 velocity=100; type continuous -> revolute
- joint robot_j2s7s300_joint_1: limit effort=40 velocity=0.6283185307179586 -> lower=-1000000 upper=1000000 effort=40 velocity=0.6283185307179586; type continuous -> revolute
- joint robot_j2s7s300_joint_3: limit effort=40 velocity=0.6283185307179586 -> lower=-1000000 upper=1000000 effort=40 velocity=0.6283185307179586; type continuous -> revolute
- joint robot_j2s7s300_joint_5: limit effort=20 velocity=0.8377580409572781 -> lower=-1000000 upper=1000000 effort=20 velocity=0.8377580409572781; type continuous -> revolute
- joint robot_j2s7s300_joint_7: limit effort=20 velocity=0.8377580409572781 -> lower=-1000000 upper=1000000 effort=20 velocity=0.8377580409572781; type continuous -> revolute
